Commit message: add dreamwaq config and mujoco resources

File: robot_lab/source/robot_lab/data/Robots/dolanga1/urdf/dolanga1.urdf (robot description, URDF)
Before this commit: robot dolanga1, 17 links, 16 joints
Joints:
- joint LF_calf_joint: limit lower=-2.82 upper=-0.8 effort=156 velocity=14 -> lower=-2.71 upper=-1.43 effort=156 velocity=14
- joint LH_calf_joint: limit lower=-2.82 upper=-0.8 effort=156 velocity=14 -> lower=-2.71 upper=-1.43 effort=156 velocity=14
- joint RF_calf_joint: limit lower=-2.82 upper=-0.8 effort=156 velocity=14 -> lower=-2.71 upper=-1.43 effort=156 velocity=14
- joint RH_calf_joint: limit lower=-2.82 upper=-0.8 effort=156 velocity=14 -> lower=-2.71 upper=-1.43 effort=156 velocity=14

Commit message: off_policy_check

File: robot_lab/source/robot_lab/data/Robots/dolanga1/urdf/dolanga1.urdf (robot description, URDF)
Before this commit: robot dolanga1, 17 links, 16 joints
Joints:
- joint LF_calf_joint: limit lower=-2.71 upper=-1.43 effort=156 velocity=14 -> lower=-2.71 upper=-1.16 effort=156 velocity=14
- joint LF_hip_joint: limit lower=-0.78 upper=0.78 effort=96 velocity=23 -> lower=-0.85 upper=0.85 effort=96 velocity=23
- joint LH_calf_joint: limit lower=-2.71 upper=-1.43 effort=156 velocity=14 -> lower=-2.71 upper=-1.16 effort=156 velocity=14
- joint LH_hip_joint: limit lower=-0.78 upper=0.78 effort=96 velocity=23 -> lower=-0.85 upper=0.85 effort=96 velocity=23
- joint RF_calf_joint: limit lower=-2.71 upper=-1.43 effort=156 velocity=14 -> lower=-2.71 upper=-1.16 effort=156 velocity=14
- joint RF_hip_joint: limit lower=-0.78 upper=0.78 effort=96 velocity=23 -> lower=-0.85 upper=0.85 effort=96 velocity=23
- joint RH_calf_joint: limit lower=-2.71 upper=-1.43 effort=156 velocity=14 -> lower=-2.71 upper=-1.16 effort=156 velocity=14
- joint RH_hip_joint: limit lower=-0.78 upper=0.78 effort=96 velocity=23 -> lower=-0.85 upper=0.85 effort=96 velocity=23
